Commit message: dependency to forked github repo

File: curtmini_piper_description/urdf/curtmini_piper.urdf.xacro (robot description, xacro)
@@ -3,5 +3,5 @@
   <!-- Reuse the complete Curt Mini model, including its ros2_control block. -->
   <xacro:include filename="$(find curt_mini)/models/curt_mini/robot.urdf.xacro" />
-  <xacro:include filename="$(find curtmini_piper_description)/urdf/piper_arm.xacro" />
+  <xacro:include filename="$(find agx_arm_urdf)/piper/urdf/piper_arm.xacro" />
   <xacro:arg name="arm_prefix" default="piper_" />
   <xacro:arg name="arm_mount_xyz" default="0 0 0.18" />
@@ -9,11 +9,15 @@
   <xacro:arg name="tcp_offset_xyz" default="0 0 0" />
   <xacro:arg name="tcp_offset_rpy" default="0 0 0" />
-  <xacro:piper_arm
-    prefix="$(arg arm_prefix)"
-    parent="chassis"
-    mount_xyz="$(arg arm_mount_xyz)"
-    mount_rpy="$(arg arm_mount_rpy)"
-    tcp_offset_xyz="$(arg tcp_offset_xyz)"
-    tcp_offset_rpy="$(arg tcp_offset_rpy)"
-  />
+  <xacro:piper_arm prefix="$(arg arm_prefix)" />
+  <joint name="$(arg arm_prefix)mount_joint" type="fixed">
+    <parent link="chassis" />
+    <child link="$(arg arm_prefix)base_link" />
+    <origin xyz="$(arg arm_mount_xyz)" rpy="$(arg arm_mount_rpy)" />
+  </joint>
+  <link name="$(arg arm_prefix)tcp_link" />
+  <joint name="$(arg arm_prefix)tcp_joint" type="fixed">
+    <parent link="$(arg arm_prefix)link6" />
+    <child link="$(arg arm_prefix)tcp_link" />
+    <origin xyz="$(arg tcp_offset_xyz)" rpy="$(arg tcp_offset_rpy)" />
+  </joint>
 </robot>

File: curtmini_piper_description/urdf/curtmini_piper_moveit.urdf.xacro (robot description, xacro)
@@ -1,5 +1,5 @@
 <?xml version="1.0"?>
 <robot xmlns:xacro="http://www.ros.org/wiki/xacro" name="curtmini_piper">
-  <xacro:include filename="$(find curtmini_piper_description)/urdf/piper_arm.xacro" />
+  <xacro:include filename="$(find agx_arm_urdf)/piper/urdf/piper_arm.xacro" />
   <xacro:arg name="simulation" default="False" />
   <xacro:arg name="arm_prefix" default="piper_" />
@@ -87,11 +87,15 @@
     <origin xyz="0.062 0 0.015" rpy="0 0 1.5707963267948966" />
   </joint>
-  <xacro:piper_arm
-    prefix="$(arg arm_prefix)"
-    parent="chassis"
-    mount_xyz="$(arg arm_mount_xyz)"
-    mount_rpy="$(arg arm_mount_rpy)"
-    tcp_offset_xyz="$(arg tcp_offset_xyz)"
-    tcp_offset_rpy="$(arg tcp_offset_rpy)"
-  />
+  <xacro:piper_arm prefix="$(arg arm_prefix)" />
+  <joint name="$(arg arm_prefix)mount_joint" type="fixed">
+    <parent link="chassis" />
+    <child link="$(arg arm_prefix)base_link" />
+    <origin xyz="$(arg arm_mount_xyz)" rpy="$(arg arm_mount_rpy)" />
+  </joint>
+  <link name="$(arg arm_prefix)tcp_link" />
+  <joint name="$(arg arm_prefix)tcp_joint" type="fixed">
+    <parent link="$(arg arm_prefix)link6" />
+    <child link="$(arg arm_prefix)tcp_link" />
+    <origin xyz="$(arg tcp_offset_xyz)" rpy="$(arg tcp_offset_rpy)" />
+  </joint>
 </robot>

File: curtmini_piper_description/urdf/piper_arm_control.urdf.xacro (robot description, xacro)
@@ -1,16 +1,20 @@
 <?xml version="1.0"?>
 <robot xmlns:xacro="http://www.ros.org/wiki/xacro" name="prefixed_piper_control">
-  <xacro:include filename="$(find curtmini_piper_description)/urdf/piper_arm.xacro" />
+  <xacro:include filename="$(find agx_arm_urdf)/piper/urdf/piper_arm.xacro" />
   <xacro:include filename="$(find curtmini_piper_description)/urdf/piper_ros2_control.xacro" />
   <xacro:arg name="arm_prefix" default="piper_" />
   <link name="$(arg arm_prefix)world" />
-  <xacro:piper_arm
-    prefix="$(arg arm_prefix)"
-    parent="$(arg arm_prefix)world"
-    mount_xyz="0 0 0"
-    mount_rpy="0 0 0"
-    tcp_offset_xyz="0 0 0"
-    tcp_offset_rpy="0 0 0"
-  />
+  <xacro:piper_arm prefix="$(arg arm_prefix)" />
+  <joint name="$(arg arm_prefix)mount_joint" type="fixed">
+    <parent link="$(arg arm_prefix)world" />
+    <child link="$(arg arm_prefix)base_link" />
+    <origin xyz="0 0 0" rpy="0 0 0" />
+  </joint>
+  <link name="$(arg arm_prefix)tcp_link" />
+  <joint name="$(arg arm_prefix)tcp_joint" type="fixed">
+    <parent link="$(arg arm_prefix)link6" />
+    <child link="$(arg arm_prefix)tcp_link" />
+    <origin xyz="0 0 0" rpy="0 0 0" />
+  </joint>
   <xacro:piper_ros2_control prefix="$(arg arm_prefix)" />
 </robot>

Commit message: add gz sim

File: curtmini_piper_description/urdf/curtmini_piper.urdf.xacro (robot description, xacro)
@@ -4,4 +4,5 @@
   <xacro:include filename="$(find curt_mini)/models/curt_mini/robot.urdf.xacro" />
   <xacro:include filename="$(find agx_arm_urdf)/piper/urdf/piper_arm.xacro" />
+  <xacro:include filename="$(find curtmini_piper_description)/urdf/piper_ros2_control.xacro" />
   <xacro:arg name="arm_prefix" default="piper_" />
   <xacro:arg name="arm_mount_xyz" default="0 0 0.18" />
@@ -21,3 +22,12 @@
     <origin xyz="$(arg tcp_offset_xyz)" rpy="$(arg tcp_offset_rpy)" />
   </joint>
+  <xacro:if value="$(arg simulation)">
+    <xacro:piper_ros2_control
+      prefix="$(arg arm_prefix)"
+      system_name="GazeboSystem"
+      hardware_plugin="gz_ros2_control/GazeboSimSystem"
+      joint2_initial_value="0.1"
+      joint3_initial_value="-0.1"
+    />
+  </xacro:if>
 </robot>

File: curtmini_piper_description/urdf/piper_arm_control.urdf.xacro (robot description, xacro)
@@ -17,4 +17,8 @@
     <origin xyz="0 0 0" rpy="0 0 0" />
   </joint>
-  <xacro:piper_ros2_control prefix="$(arg arm_prefix)" />
+  <xacro:piper_ros2_control
+    prefix="$(arg arm_prefix)"
+    system_name="FakeSystem"
+    hardware_plugin="mock_components/GenericSystem"
+  />
 </robot>

File: curtmini_piper_description/urdf/piper_ros2_control.xacro (robot description, xacro)
@@ -1,24 +1,42 @@
 <?xml version="1.0"?>
 <robot xmlns:xacro="http://www.ros.org/wiki/xacro">
-  <xacro:macro name="piper_ros2_control" params="prefix">
-    <ros2_control name="${prefix}FakeSystem" type="system">
+  <xacro:macro
+    name="piper_ros2_control"
+    params="
+      prefix
+      system_name
+      hardware_plugin
+      joint2_initial_value:=0.0
+      joint3_initial_value:=0.0
+    "
+  >
+    <ros2_control name="${prefix}${system_name}" type="system">
       <hardware>
-        <plugin>mock_components/GenericSystem</plugin>
+        <plugin>${hardware_plugin}</plugin>
       </hardware>
-      <xacro:macro name="piper_control_joint" params="joint_name">
+      <xacro:macro
+        name="piper_control_joint"
+        params="joint_name initial_value"
+      >
         <joint name="${prefix}${joint_name}">
           <command_interface name="position" />
           <state_interface name="position">
-            <param name="initial_value">0.0</param>
+            <param name="initial_value">${initial_value}</param>
           </state_interface>
           <state_interface name="velocity" />
         </joint>
       </xacro:macro>
-      <xacro:piper_control_joint joint_name="joint1" />
-      <xacro:piper_control_joint joint_name="joint2" />
-      <xacro:piper_control_joint joint_name="joint3" />
-      <xacro:piper_control_joint joint_name="joint4" />
-      <xacro:piper_control_joint joint_name="joint5" />
-      <xacro:piper_control_joint joint_name="joint6" />
+      <xacro:piper_control_joint joint_name="joint1" initial_value="0.0" />
+      <xacro:piper_control_joint
+        joint_name="joint2"
+        initial_value="${joint2_initial_value}"
+      />
+      <xacro:piper_control_joint
+        joint_name="joint3"
+        initial_value="${joint3_initial_value}"
+      />
+      <xacro:piper_control_joint joint_name="joint4" initial_value="0.0" />
+      <xacro:piper_control_joint joint_name="joint5" initial_value="0.0" />
+      <xacro:piper_control_joint joint_name="joint6" initial_value="0.0" />
     </ros2_control>
   </xacro:macro>

Commit message: sync to new curt_mini: curtmini models lives in curt_mini_description

File: curtmini_piper_description/urdf/curtmini_piper.urdf.xacro (robot description, xacro)
@@ -2,5 +2,5 @@
 <robot xmlns:xacro="http://www.ros.org/wiki/xacro" name="curtmini_piper">
   <!-- Reuse the complete Curt Mini model, including its ros2_control block. -->
-  <xacro:include filename="$(find curt_mini)/models/curt_mini/robot.urdf.xacro" />
+  <xacro:include filename="$(find curt_mini_description)/models/curt_mini/robot.urdf.xacro" />
   <xacro:include filename="$(find agx_arm_urdf)/piper/urdf/piper_arm.xacro" />
   <xacro:include filename="$(find curtmini_piper_description)/urdf/piper_ros2_control.xacro" />

File: curtmini_piper_description/urdf/curtmini_piper_moveit.urdf.xacro (robot description, xacro)
@@ -12,5 +12,5 @@
     <visual>
       <geometry>
-        <mesh filename="package://curt_mini/models/curt_mini/meshes/base_link.STL" />
+        <mesh filename="package://curt_mini_description/models/curt_mini/meshes/base_link.STL" />
       </geometry>
       <material name="curt_mini_body">
@@ -34,5 +34,5 @@
       <visual>
         <geometry>
-          <mesh filename="package://curt_mini/models/curt_mini/meshes/${mesh}" />
+          <mesh filename="package://curt_mini_description/models/curt_mini/meshes/${mesh}" />
         </geometry>
         <material name="curt_mini_body" />

Commit message: add curtmini_piper_description/config/geometry.yaml : arm position, tcp offset and lidar mount position

File: curtmini_piper_description/urdf/curtmini_piper.urdf.xacro (robot description, xacro)
@@ -6,12 +6,13 @@
   <xacro:include filename="$(find curtmini_piper_description)/urdf/piper_ros2_control.xacro" />
   <xacro:include filename="$(find curtmini_piper_description)/urdf/hokuyo_utm_30lx_ew.xacro" />
+  <xacro:include filename="$(find curtmini_piper_description)/urdf/geometry.xacro" />
   <xacro:arg name="arm_prefix" default="piper_" />
-  <xacro:arg name="arm_mount_xyz" default="0 0 0.18" />
-  <xacro:arg name="arm_mount_rpy" default="0 0 0" />
-  <xacro:arg name="tcp_offset_xyz" default="0 0 0" />
-  <xacro:arg name="tcp_offset_rpy" default="0 0 0" />
   <xacro:arg name="use_hokuyo" default="False" />
-  <xacro:arg name="hokuyo_mount_xyz" default="0.25 0 0.20" />
-  <xacro:arg name="hokuyo_mount_rpy" default="0 0 0" />
+  <xacro:arg name="piper_joint1_initial_value" default="0.0" />
+  <xacro:arg name="piper_joint2_initial_value" default="0.1" />
+  <xacro:arg name="piper_joint3_initial_value" default="-0.1" />
+  <xacro:arg name="piper_joint4_initial_value" default="0.0" />
+  <xacro:arg name="piper_joint5_initial_value" default="0.0" />
+  <xacro:arg name="piper_joint6_initial_value" default="-1.95" />
   <xacro:arg
     name="piper_joint_limits_file"
@@ -23,5 +24,5 @@
     <parent link="chassis" />
     <child link="$(arg arm_prefix)base_link" />
-    <origin xyz="$(arg arm_mount_xyz)" rpy="$(arg arm_mount_rpy)" />
+    <origin xyz="${arm_mount_xyz}" rpy="${arm_mount_rpy}" />
   </joint>
   <link name="$(arg arm_prefix)tcp_link" />
@@ -29,11 +30,11 @@
     <parent link="$(arg arm_prefix)link6" />
     <child link="$(arg arm_prefix)tcp_link" />
-    <origin xyz="$(arg tcp_offset_xyz)" rpy="$(arg tcp_offset_rpy)" />
+    <origin xyz="${tcp_offset_xyz}" rpy="${tcp_offset_rpy}" />
   </joint>
   <xacro:if value="$(arg use_hokuyo)">
     <xacro:hokuyo_utm_30lx_ew
       parent="chassis"
-      xyz="$(arg hokuyo_mount_xyz)"
-      rpy="$(arg hokuyo_mount_rpy)"
+      xyz="${hokuyo_mount_xyz}"
+      rpy="${hokuyo_mount_rpy}"
     />
   </xacro:if>
@@ -43,7 +44,10 @@
       system_name="GazeboSystem"
       hardware_plugin="gz_ros2_control/GazeboSimSystem"
-      joint2_initial_value="0.1"
-      joint3_initial_value="-0.1"
-      joint6_initial_value="-1.95"
+      joint1_initial_value="$(arg piper_joint1_initial_value)"
+      joint2_initial_value="$(arg piper_joint2_initial_value)"
+      joint3_initial_value="$(arg piper_joint3_initial_value)"
+      joint4_initial_value="$(arg piper_joint4_initial_value)"
+      joint5_initial_value="$(arg piper_joint5_initial_value)"
+      joint6_initial_value="$(arg piper_joint6_initial_value)"
     />
   </xacro:if>

File: curtmini_piper_description/urdf/curtmini_piper_moveit.urdf.xacro (robot description, xacro)
@@ -3,13 +3,8 @@
   <xacro:include filename="$(find agx_arm_urdf)/piper/urdf/piper_arm.xacro" />
   <xacro:include filename="$(find curtmini_piper_description)/urdf/hokuyo_utm_30lx_ew.xacro" />
+  <xacro:include filename="$(find curtmini_piper_description)/urdf/geometry.xacro" />
   <xacro:arg name="simulation" default="False" />
   <xacro:arg name="arm_prefix" default="piper_" />
-  <xacro:arg name="arm_mount_xyz" default="0 0 0.18" />
-  <xacro:arg name="arm_mount_rpy" default="0 0 0" />
-  <xacro:arg name="tcp_offset_xyz" default="0 0 0" />
-  <xacro:arg name="tcp_offset_rpy" default="0 0 0" />
   <xacro:arg name="use_hokuyo" default="False" />
-  <xacro:arg name="hokuyo_mount_xyz" default="0.25 0 0.20" />
-  <xacro:arg name="hokuyo_mount_rpy" default="0 0 0" />
   <xacro:arg
     name="piper_joint_limits_file"
@@ -100,5 +95,5 @@
     <parent link="chassis" />
     <child link="$(arg arm_prefix)base_link" />
-    <origin xyz="$(arg arm_mount_xyz)" rpy="$(arg arm_mount_rpy)" />
+    <origin xyz="${arm_mount_xyz}" rpy="${arm_mount_rpy}" />
   </joint>
   <link name="$(arg arm_prefix)tcp_link" />
@@ -106,11 +101,11 @@
     <parent link="$(arg arm_prefix)link6" />
     <child link="$(arg arm_prefix)tcp_link" />
-    <origin xyz="$(arg tcp_offset_xyz)" rpy="$(arg tcp_offset_rpy)" />
+    <origin xyz="${tcp_offset_xyz}" rpy="${tcp_offset_rpy}" />
   </joint>
   <xacro:if value="$(arg use_hokuyo)">
     <xacro:hokuyo_utm_30lx_ew
       parent="chassis"
-      xyz="$(arg hokuyo_mount_xyz)"
-      rpy="$(arg hokuyo_mount_rpy)"
+      xyz="${hokuyo_mount_xyz}"
+      rpy="${hokuyo_mount_rpy}"
     />
   </xacro:if>

File: curtmini_piper_description/urdf/piper_ros2_control.xacro (robot description, xacro)
@@ -7,6 +7,9 @@
       system_name
       hardware_plugin
+      joint1_initial_value:=0.0
       joint2_initial_value:=0.0
       joint3_initial_value:=0.0
+      joint4_initial_value:=0.0
+      joint5_initial_value:=0.0
       joint6_initial_value:=0.0
     "
@@ -28,5 +31,8 @@
         </joint>
       </xacro:macro>
-      <xacro:piper_control_joint joint_name="joint1" initial_value="0.0" />
+      <xacro:piper_control_joint
+        joint_name="joint1"
+        initial_value="${joint1_initial_value}"
+      />
       <xacro:piper_control_joint
         joint_name="joint2"
@@ -37,6 +43,12 @@
         initial_value="${joint3_initial_value}"
       />
-      <xacro:piper_control_joint joint_name="joint4" initial_value="0.0" />
-      <xacro:piper_control_joint joint_name="joint5" initial_value="0.0" />
+      <xacro:piper_control_joint
+        joint_name="joint4"
+        initial_value="${joint4_initial_value}"
+      />
+      <xacro:piper_control_joint
+        joint_name="joint5"
+        initial_value="${joint5_initial_value}"
+      />
       <xacro:piper_control_joint
         joint_name="joint6"

Commit message: add curtmini_sensor for two cameras (here d435i)

File: curtmini_piper_description/urdf/curtmini_piper.urdf.xacro (robot description, xacro)
@@ -6,4 +6,5 @@
   <xacro:include filename="$(find curtmini_piper_description)/urdf/piper_ros2_control.xacro" />
   <xacro:include filename="$(find curtmini_piper_description)/urdf/hokuyo_utm_30lx_ew.xacro" />
+  <xacro:include filename="$(find curtmini_piper_description)/urdf/d435i_body.xacro" />
   <xacro:include filename="$(find curtmini_piper_description)/urdf/geometry.xacro" />
   <xacro:arg name="arm_prefix" default="piper_" />
@@ -32,4 +33,8 @@
     <origin xyz="${tcp_offset_xyz}" rpy="${tcp_offset_rpy}" />
   </joint>
+  <xacro:d435i_body name="base_camera" parent="chassis"
+    xyz="${base_camera_mount_xyz}" rpy="${base_camera_mount_rpy}" />
+  <xacro:d435i_body name="tool_camera" parent="$(arg arm_prefix)tcp_link"
+    xyz="${tool_camera_mount_xyz}" rpy="${tool_camera_mount_rpy}" />
   <xacro:if value="$(arg use_hokuyo)">
     <xacro:hokuyo_utm_30lx_ew

File: curtmini_piper_description/urdf/curtmini_piper_moveit.urdf.xacro (robot description, xacro)
@@ -3,4 +3,5 @@
   <xacro:include filename="$(find agx_arm_urdf)/piper/urdf/piper_arm.xacro" />
   <xacro:include filename="$(find curtmini_piper_description)/urdf/hokuyo_utm_30lx_ew.xacro" />
+  <xacro:include filename="$(find curtmini_piper_description)/urdf/d435i_body.xacro" />
   <xacro:include filename="$(find curtmini_piper_description)/urdf/geometry.xacro" />
   <xacro:arg name="simulation" default="False" />
@@ -103,4 +104,8 @@
     <origin xyz="${tcp_offset_xyz}" rpy="${tcp_offset_rpy}" />
   </joint>
+  <xacro:d435i_body name="base_camera" parent="chassis"
+    xyz="${base_camera_mount_xyz}" rpy="${base_camera_mount_rpy}" />
+  <xacro:d435i_body name="tool_camera" parent="$(arg arm_prefix)tcp_link"
+    xyz="${tool_camera_mount_xyz}" rpy="${tool_camera_mount_rpy}" />
   <xacro:if value="$(arg use_hokuyo)">
     <xacro:hokuyo_utm_30lx_ew

File: curtmini_piper_description/urdf/geometry.xacro (robot description, xacro)
@@ -11,3 +11,7 @@
   <xacro:property name="hokuyo_mount_xyz" value="${geometry['lidar_mount_on_base']['position']['x']} ${geometry['lidar_mount_on_base']['position']['y']} ${geometry['lidar_mount_on_base']['position']['z']}" />
   <xacro:property name="hokuyo_mount_rpy" value="${geometry['lidar_mount_on_base']['rotation']['r']} ${geometry['lidar_mount_on_base']['rotation']['p']} ${geometry['lidar_mount_on_base']['rotation']['y']}" />
+  <xacro:property name="base_camera_mount_xyz" value="${geometry['base_camera_mount']['position']['x']} ${geometry['base_camera_mount']['position']['y']} ${geometry['base_camera_mount']['position']['z']}" />
+  <xacro:property name="base_camera_mount_rpy" value="${geometry['base_camera_mount']['rotation']['r']} ${geometry['base_camera_mount']['rotation']['p']} ${geometry['base_camera_mount']['rotation']['y']}" />
+  <xacro:property name="tool_camera_mount_xyz" value="${geometry['tool_camera_mount']['position']['x']} ${geometry['tool_camera_mount']['position']['y']} ${geometry['tool_camera_mount']['position']['z']}" />
+  <xacro:property name="tool_camera_mount_rpy" value="${geometry['tool_camera_mount']['rotation']['r']} ${geometry['tool_camera_mount']['rotation']['p']} ${geometry['tool_camera_mount']['rotation']['y']}" />
 </robot>
